Commit message: 250125

File: urdf/yixiuge_d435i.xacro (robot description, xacro)
@@ -55,5 +55,5 @@
 				<geometry>
 					<!-- <box size="0.01 0.01 0.01"/> -->
-					<mesh filename="package://robot_sim2/urdf/meshes/d435i.dae" />
+					<mesh filename="package://ros2_sim/urdf/meshes/d435i.dae" />
 				</geometry>
 			</collision>
@@ -66,5 +66,5 @@
 					<!-- <mesh filename="package://robot_sim_demo/models/meshes/xtion_pro_camera.dae" /> -->
 					<!-- <mesh filename="package://robot_sim_demo/models/meshes/kinect.dae" /> -->
-					<mesh filename="package://robot_sim2/urdf/meshes/d435i.dae" />
+					<mesh filename="package://ros2_sim/urdf/meshes/d435i.dae" />
 				</geometry>
 				<material name="">

File: urdf/yixiuge_d435i_gazebo.xacro (robot description, xacro)
@@ -3,5 +3,5 @@
   <xacro:property name="M_PI" value="3.141592653589793"/>
   <link name="world" />
-  <xacro:include filename="$(find robot_sim2)/urdf/yixiuge_d435i.xacro" />
+  <xacro:include filename="$(find ros2_sim)/urdf/yixiuge_d435i.xacro" />
   <xacro:yixiuge_d435i />
   <joint name="yixiuge_d435i_base_joint" type="fixed">
